File: leds.kicad_pcb (KiCad board)
At the start: 2 copper layers, 48.5 x 37.5 mm, 7 parts, among them SW1 SW_Push, SW3 SW_Push

Commit message: new thing
Parts:
- removed D2: LED, LED_THT:LED_D5.0mm
- removed R2: R, Resistor_THT:R_Axial_DIN0207_L6.3mm_D2.5mm_P7.62mm_Horizontal
- added G***: LOGO, LOGO, F.Cu at (166.5, 115.0)
- added G***: LOGO, LOGO, F.Cu at (132.0, 117.0)
- added Q1: NPN, Package_TO_SOT_THT:TO-92L_HandSolder, F.Cu at (154.2, 110.0)
- added Q2: NPN, Package_TO_SOT_THT:TO-92L_HandSolder, F.Cu at (141.2, 110.0)
- added R3: R, Resistor_THT:R_Axial_DIN0207_L6.3mm_D2.5mm_P7.62mm_Horizontal, F.Cu at (127.4, 109.5)
- added R4: R, Resistor_THT:R_Axial_DIN0207_L6.3mm_D2.5mm_P7.62mm_Horizontal, F.Cu at (127.7, 103.5)
- moved SW3 35.3 mm to (127.8, 92.8)
- moved SW1 35.3 mm to (163.8, 92.8)
- moved R1 35.0 mm to (163.2, 103.5)
- moved D1 17.0 mm to (147.7, 109.5)
- moved BT1 1.05 mm to (149.1, 95.4)
Connections:
- R1 pad 1: Net-(D1-K) -> Net-(BT1-+)
- R1 pad 2: Net-(BT1--) -> Net-(D1-A)
- SW1 pad 2: Net-(D1-A) -> Net-(R4-Pad1)
Routing:
- net Net-(BT1-+): track 53.2 -> 0.00 mm
- net Net-(BT1--): track 40.5 -> 0.00 mm
- net Net-(D2-K): track 31.1 -> 0.00 mm
- net Net-(R3-Pad1): track 18.1 -> 0.00 mm
- net Net-(D1-A): track 17.0 -> 0.00 mm
- net Net-(D1-K): track 6.55 -> 0.00 mm
Other:
- outline, holes or cut-outs redrawn
- board text added: "Made with Skill Issues by Heinrich"
